File: stepper.kicad_sch (KiCad schematic)
At the start: 32 parts, among them U6 TMC2209-LA, U7 TMC2209-LA

Commit message: added power button
Parts:
- renumbered C39 to C34, C40 to C35, C41 to C36, C42 to C37, C43 to C38, C44 to C39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
